Commit message: Update robotable_with_gripper.urdf
better...

File: gym_robotable/envs/robotable_with_gripper.urdf (robot description, URDF)
Before this commit: robot table, 8 links, 7 joints
Links:
- link neck_1: mass 1 -> 1.618; geometry collision box size=0.1 0.1 1.618; visual box size=0.1 0.1 1.618
- link neck_2: geometry collision box size=0.1 0.1 1; visual box size=0.1 0.1 1
- link neck_3: geometry collision box size=0.1 0.1 0.618; visual box size=0.1 0.1 0.618
Joints:
- joint gripper_joint_1: child shoulder -> neck_1; origin xyz=0 0 1 rpy=0 0 0 -> xyz=0 0.618 1.1 rpy=3 0 0
- joint gripper_joint_2: origin xyz=0 0 0.8 rpy=0 0 0 -> xyz=0 0 -1.618 rpy=-1 0 0
- joint gripper_joint_3: origin xyz=0 0 0.6 rpy=0 0 0 -> xyz=0 0 -1 rpy=0 0 0

Commit message: Update robotable_with_gripper.urdf
a bit better motor positions, though still a bit off.

File: gym_robotable/envs/robotable_with_gripper.urdf (robot description, URDF)
Before this commit: robot table, 8 links, 7 joints
Links:
- added link neck_0, mass 1.618; collision cylinder length=0.1 radius=0.1; visual cylinder length=0.1 radius=0.1
Joints:
- added joint gripper_joint_0: type revolute, parent chassis, child neck_0, origin xyz=0 0.618 1.1 rpy=0 0 0, axis 0 0 1, limit lower=-1.57. upper=1.57 effort=10.0 velocity=1000.0
- joint gripper_joint_1: origin xyz=0 0.618 1.1 rpy=3 0 0 -> xyz=0 0 0 rpy=3 0 0; parent chassis -> neck_0
- joint gripper_joint_2: origin xyz=0 0 -1.618 rpy=-1 0 0 -> xyz=0 0 -1.718 rpy=-1 0 0

Commit message: update for gripper code

File: gym_robotable/envs/robotable_with_gripper.urdf (robot description, URDF)
Before this commit: robot table, 8 links, 7 joints
Links:
- added link neck_0, mass 1.618; collision cylinder length=0.1 radius=0.1; visual cylinder length=0.1 radius=0.1
- link neck_1: mass 1 -> 1.618; geometry collision box size=0.1 0.1 1.618; visual box size=0.1 0.1 1.618
- link neck_2: geometry collision box size=0.1 0.1 1; visual box size=0.1 0.1 1
- link neck_3: geometry collision box size=0.1 0.1 0.618; visual box size=0.1 0.1 0.618
Joints:
- added joint gripper_joint_0: type revolute, parent chassis, child neck_0, origin xyz=0 0.618 1.1 rpy=0 0 0, axis 0 0 1, limit lower=-1.57. upper=1.57 effort=10.0 velocity=1000.0
- joint gripper_joint_1: child shoulder -> neck_1; origin xyz=0 0 1 rpy=0 0 0 -> xyz=0 0 0 rpy=2.7 0 0; parent chassis -> neck_0
- joint gripper_joint_2: origin xyz=0 0 0.8 rpy=0 0 0 -> xyz=0 0 -1.718 rpy=-0.9 0 0
- joint gripper_joint_3: origin xyz=0 0 0.6 rpy=0 0 0 -> xyz=0 0 -1 rpy=0 0 0
